File: kiCAD/tremolo_guitar_pedal/tremolo_guitar_pedal.kicad_sch (KiCad schematic)
At the start: 53 parts, among them CN3 NUCLEO-L432KC, CN4 NUCLEO-L432KC, J1 1/4" Mono Jack, J2 1/4" Mono Jack, J3 UPduino v3.1, J4 Barrel_Jack, J5 UPduino v3.1, SW1 3PDT Footswitch, SW2 3PDT Footswitch, SW3 3PDT Footswitch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

Commit message: schematic update
Parts:
- removed CN3: NUCLEO-L432KC, symbol Connector_Generic:Conn_01x02
- removed CN4: NUCLEO-L432KC, symbol Connector_Generic:Conn_01x01
- removed J3: UPduino v3.1, symbol Connector_Generic:Conn_01x02
- removed U2: PCM5102, Package_SO:TSSOP-28_4.4x9.7mm_P0.65mm, symbol Audio:PCM5122PW
- removed U5: STM32L432KCUx, Package_DFN_QFN:QFN-32-1EP_5x5mm_P0.5mm_EP3.45x3.45mm, symbol MCU_ST_STM32L4:STM32L432KCUx
- removed U6: ICE40UP5K-SG48ITR, Package_DFN_QFN:QFN-48-1EP_7x7mm_P0.5mm_EP5.6x5.6mm, symbol FPGA_Lattice:ICE40UP5K-SG48ITR
- removed depth, mix: 10k, symbol Device:R_Potentiometer
- removed speed: 10k, log, symbol Device:R_Potentiometer
- added U4: NUCLEO-LxxxKx, E155_Footprints:NUCLEO-32, symbol E155_Symbols:NUCLEO-LxxxKx
- added U5: PCM5102, Package_SO:TSSOP-28_4.4x9.7mm_P0.65mm, symbol Audio:PCM5122PW
- added U7: UPduino_v3.1, E155_Footprints:UPduino_v3.1, symbol E155_Symbols:UPduino_v3.1
Connections:
- net +3.3V: now also U5.1 (VIN)
- net AGND: now also U5.9 (AGND)
- net DGND: now also U5.2 (GND)
- net FPGA_FS: now also J5.44 (P20), U5.3 (WSEL); no longer J5.33 (P6)
- net FPGA_SCK: now also J5.38 (13), U5.5 (BCK); no longer J5.31 (P4)
- net FPGA_SD: now also J5.40 (P12), U5.4 (DIN); no longer J5.30 (P3)
- net GND: now also U4.29 (GND), U4.4 (GND), U7.1 (GND), U7.10 (GND), U7.42 (GND)
- net P11: now also U7.35 (GPIO_11)
- net P19: now also U7.37 (GPIO_19)
- net P31: now also U7.17 (GPIO_31)
- net P32: now also U7.15 (GPIO_32)
- net P35: now also U7.16 (GPIO_35)
- net P37: now also U7.18 (GPIO_37)
- net P4: now also U7.31 (GPIO_4)
- net P6: now also U7.33 (GPIO_6)
- net at R10.1: now also U5.8 (Lout)
- net ADC1_IN5: no longer names the net of C6.2, U2.6 (-), U2.7
- new net: U4.1 (D1/PA9/TX1), U7.12 (GPIO_25)
- new net: U4.12 (D9/PA8), U7.27 (GPIO_47)
- new net: U4.2 (D0/PA10/RX1), U7.11 (GPIO_23)
- new net FPGA_+3V3: U7.9 (+3.3V)
- new net FPGA_+5: U7.8 (+5V)
- new net MCU_+5V: U4.27 (+5V)
- new net MCU_AREF: U4.18 (AREF)
- new net P12: U7.40 (GPIO_12)
- new net P13: U7.38 (GPIO_13)
- new net P20: U7.44 (GPIO_20)
- new net P28: U7.24 (GPIO_28)
- new net P38: U7.23 (GPIO_38)
- new net P43: U7.20 (GPIO_43)
- new net P47: U7.4 (DONE)
- new net PA10: U4.21 (A2/PA3)
- new net PA8: U4.19 (A0/PA0)
- new net PA9: U4.20 (A1/PA1)
- new net ~{FPGA_RESET}: U7.3 (~{RST})
- new net ~{MCU_RESET}: U4.28 (~{RESET}), U4.3 (~{RESET})
- no-connect marks 1 -> 9
Other:
- note added: "SCLK"
- note added: "SD"
- note added: "STM32 MCU"
- note added: "UP5K FPGA"
- note added: "WS"
- note removed: "0.1x attenuation output buffer"
- note removed: "Effect Potentiometers"
- note removed: "I2S between MCU and FPGA"
- note removed: "PA9 for FS"
- note removed: "change these"
- note removed: "the coupling cap value depends on the input impedance of the guitar amp"
- note removed: "these FPGA pins are arbitrary"
- note removed: "these will go to MCU pins"
- moved on the sheet: C1, C2, U3A
